Commit message: working gazebo setup from one launchfile, no control yet

File: src/m1u_description/urdf/m1-u_combine.urdf (robot description, URDF)
Before this commit: robot m1u_description, 7 links, 6 joints
Links:
- added link world
Joints:
- added joint world_to_base_link_fixed_joint: type fixed, parent world, child base_link, origin xyz=0 0 0 rpy=0 0 0
